File: RS232toTTL.sch (KiCad schematic (older format))
At the start: 15 parts, among them J1 DB9, P1 CONN_01X04, Q1 2N7002, Q2 PNP-BC857

Commit message: Routing PCB
Connections:
- net GND: now also P1.1 (P1); no longer P1.4 (P4)
- net VCC: now also P1.4 (P4); no longer P1.1 (P1)
- net at D2.1 (K), R5.2: now also P1.3 (P3); no longer P1.2 (P2)
- net at D3.1 (K), Q1.3 (D), R3.2: now also P1.2 (P2); no longer P1.3 (P3)
Other:
- note added: "or BSS138"
Changed lines of the file:
@@
 F 3 "" H 7700 3200 50  0000 C CNN
 	1    7700 3200
-	1    0    0    -1
+	1    0    0    1
 $EndComp
 $Comp
@@
 Wire Wire Line
 	3800 3025 3800 2525
+Text Notes 5525 4000 0    60   ~ 0
+or BSS138
 $EndSCHEMATC
